File: proto_array.sch (KiCad schematic (older format))
At the start: 60 parts, among them P1 CONN_01X03, P2 CONN_01X03, P3 CONN_01X03, P4 CONN_01X03, P5 CONN_01X03, U1 ADS131E08, U2 BEAGLEBONEBLACK

Commit message: Eliminated the headers for SPI interface to make PCB single layer.
Signed-off-by: Chamon <[luizchamon@gmail.com>
Parts:
- removed P1, P2, P3, P4: CONN_01X03, Pin_Headers:Pin_Header_Straight_1x03, symbol CONN_01X03
- renumbered P5 to P1
Connections:
- wire segments 249 -> 235
Changed lines of the file:
@@
 Text Label 8600 1050 2    60   ~ 0
 PRU1_2
-Text Label 9100 800  0    60   ~ 0
+Text Label 8600 1200 2    60   ~ 0
 PRU1_5
-Text Label 9100 1200 0    60   ~ 0
+Text Label 8600 1300 2    60   ~ 0
 PRU1_3
-Text Label 9100 1600 0    60   ~ 0
+Text Label 8600 1400 2    60   ~ 0
 PRU1_7
-Text Label 9100 2000 0    60   ~ 0
+Text Label 8600 1500 2    60   ~ 0
 PRU1_1
 Text Label 8600 2050 2    60   ~ 0
@@
 	8150 1050 8600 1050
 Wire Wire Line
-	8150 1200 8850 1200
-Wire Wire Line
-	8150 1400 8850 1400
-Wire Wire Line
-	8150 1500 8800 1500
+	8150 1200 8600 1200
+Wire Wire Line
+	8150 1400 8600 1400
+Wire Wire Line
+	8150 1500 8600 1500
 Wire Wire Line
 	8600 2050 8150 2050
@@
 BBB_5V
 $Comp
-L CONN_01X03 P5
+L CONN_01X03 P1
 U 1 1 5566C302
 P 1050 3300
-F 0 "P5" H 1050 3500 50  0000 C CNN
+F 0 "P1" H 1050 3500 50  0000 C CNN
 F 1 "CONN_01X03" V 1150 3300 50  0001 C CNN
 F 2 "Pin_Headers:Pin_Header_Straight_1x03" H 1050 3300 60  0001 C CNN
@@
 Text Notes 4000 4350 0    60   ~ 0
 Place capacitors as close as possible to BBB headers.
-Text Label 9100 1000 0    60   ~ 0
-SPI0_CS
-Text Label 9000 2200 0    60   ~ 0
-SPI0_MISO
-Text Label 9000 1800 0    60   ~ 0
-SPI0_MOSI
-Text Label 9050 1400 0    60   ~ 0
-SPI0_CLK
-$Comp
-L CONN_01X03 P1
-U 1 1 556688D0
-P 9700 900
-F 0 "P1" H 9700 1100 50  0000 C CNN
-F 1 "CONN_01X03" V 9800 900 50  0001 C CNN
-F 2 "Pin_Headers:Pin_Header_Straight_1x03" H 9700 900 60  0001 C CNN
-F 3 "" H 9700 900 60  0000 C CNN
-	1    9700 900
-	1    0    0    -1
-$EndComp
-$Comp
-L CONN_01X03 P2
-U 1 1 55669581
-P 9700 1300
-F 0 "P2" H 9700 1500 50  0000 C CNN
-F 1 "CONN_01X03" V 9800 1300 50  0001 C CNN
-F 2 "Pin_Headers:Pin_Header_Straight_1x03" H 9700 1300 60  0001 C CNN
-F 3 "" H 9700 1300 60  0000 C CNN
-	1    9700 1300
-	1    0    0    -1
-$EndComp
-$Comp
-L CONN_01X03 P3
-U 1 1 55669C69
-P 9700 1700
-F 0 "P3" H 9700 1900 50  0000 C CNN
-F 1 "CONN_01X03" V 9800 1700 50  0001 C CNN
-F 2 "Pin_Headers:Pin_Header_Straight_1x03" H 9700 1700 60  0001 C CNN
-F 3 "" H 9700 1700 60  0000 C CNN
-	1    9700 1700
-	1    0    0    -1
-$EndComp
-$Comp
-L CONN_01X03 P4
-U 1 1 5566BE22
-P 9700 2100
-F 0 "P4" H 9700 2300 50  0000 C CNN
-F 1 "CONN_01X03" V 9800 2100 50  0001 C CNN
-F 2 "Pin_Headers:Pin_Header_Straight_1x03" H 9700 2100 60  0001 C CNN
-F 3 "" H 9700 2100 60  0000 C CNN
-	1    9700 2100
-	1    0    0    -1
-$EndComp
-Wire Wire Line
-	9100 1000 9500 1000
-Wire Wire Line
-	9100 800  9500 800
-Wire Wire Line
-	9500 900  8850 900
-Wire Wire Line
-	8850 900  8850 1200
-Wire Wire Line
-	9500 2100 8800 2100
-Wire Wire Line
-	8800 2100 8800 1500
-Wire Wire Line
-	9500 1700 8850 1700
-Wire Wire Line
-	8850 1700 8850 1400
-Wire Wire Line
-	9500 1200 9100 1200
-Wire Wire Line
-	9500 1400 9050 1400
-Wire Wire Line
-	8150 1300 9500 1300
-Wire Wire Line
-	9500 1600 9100 1600
-Wire Wire Line
-	9500 1800 9000 1800
-Wire Wire Line
-	9500 2000 9100 2000
-Wire Wire Line
-	9500 2200 9000 2200
 Wire Notes Line
 	9900 2600 9900 550
@@
 Wire Wire Line
 	12450 5750 12900 5750
+Wire Wire Line
+	8150 1300 8600 1300
 $EndSCHEMATC

Commit message: * Fix PRU connections on the schematic * Reduce microphone tracks to fit ground plane * Remove fiducials from ADC IC
Signed-off-by: Chamon <[luizchamon@gmail.com>
Parts:
- U1: footprint micarray:LQFP-64_12x12_Pitch0.5mm -> micarray:LQFP-64_12x12_Pitch0.5mm_NoFid
Changed lines of the file:
@@
 F 0 "U1" H 6150 7000 60  0000 C CNN
 F 1 "ADS131E08" H 6150 5150 60  0000 C CNN
-F 2 "micarray:LQFP-64_12x12_Pitch0.5mm" H 6000 6650 60  0001 C CNN
+F 2 "micarray:LQFP-64_12x12_Pitch0.5mm_NoFid" H 6000 6650 60  0001 C CNN
 F 3 "" H 6000 6650 60  0000 C CNN
 	1    6150 6100
@@
 F 0 "U1" H 950 2150 60  0000 C CNN
 F 1 "ADS131E08" H 900 1100 60  0000 C CNN
-F 2 "micarray:LQFP-64_12x12_Pitch0.5mm" H 1750 2200 60  0001 C CNN
+F 2 "micarray:LQFP-64_12x12_Pitch0.5mm_NoFid" H 1750 2200 60  0001 C CNN
 F 3 "" H 1750 2200 60  0000 C CNN
 	2    1900 1650
@@
 F 0 "U1" H 7600 2300 60  0000 C CNN
 F 1 "ADS131E08" H 7600 750 60  0000 C CNN
-F 2 "micarray:LQFP-64_12x12_Pitch0.5mm" H 7450 2100 60  0001 C CNN
+F 2 "micarray:LQFP-64_12x12_Pitch0.5mm_NoFid" H 7450 2100 60  0001 C CNN
 F 3 "" H 7450 2100 60  0000 C CNN
 	3    7600 1550
@@
 	11050 4850 10500 4850
 Text Label 8600 950  2    60   ~ 0
+PRU1_4
+Text Label 8600 1050 2    60   ~ 0
+PRU1_1
+Text Label 8600 1200 2    60   ~ 0
+PRU1_7
+Text Label 8600 1300 2    60   ~ 0
+PRU1_5
+Text Label 8600 1400 2    60   ~ 0
 PRU1_0
-Text Label 8600 1050 2    60   ~ 0
+Text Label 8600 1500 2    60   ~ 0
+PRU1_3
+Text Label 8600 2050 2    60   ~ 0
 PRU1_2
-Text Label 8600 1200 2    60   ~ 0
-PRU1_5
-Text Label 8600 1300 2    60   ~ 0
-PRU1_3
-Text Label 8600 1400 2    60   ~ 0
-PRU1_7
-Text Label 8600 1500 2    60   ~ 0
-PRU1_1
-Text Label 8600 2050 2    60   ~ 0
-PRU1_4
 Wire Wire Line
 	8150 950  8600 950

Commit message: Final PCB with one airwire.
Signed-off-by: Chamon <[luizchamon@gmail.com>
Parts:
- removed TP2: TESTPOINT, Measurement_Points:Measurement_Point_Round-SMD-Pad_Big, symbol TESTPOINT
Connections:
- wire segments 235 -> 234
Changed lines of the file:
@@
 Text Notes 800  4850 0    60   ~ 0
 ERC warnings relative to power output pins\nbeing connected to bidirectional pins on the\nBBB headers can safely be ignored.
-$Comp
-L TESTPOINT TP2
-U 1 1 5567DDB5
-P 2550 700
-F 0 "TP2" H 2800 700 40  0000 C CNN
-F 1 "TESTPOINT" H 2600 600 40  0001 C CNN
-F 2 "Measurement_Points:Measurement_Point_Round-SMD-Pad_Big" H 2750 700 60  0001 C CNN
-F 3 "" H 2750 700 60  0000 C CNN
-	1    2550 700
-	1    0    0    -1
-$EndComp
-Wire Wire Line
-	2500 700  2550 700
 Wire Wire Line
 	5550 950  5550 850

Commit message: * Add ADC footprint without fiducials * Remove unused pin headers from BBB * Modify eletret footprint
Signed-off-by: Chamon <[luizchamon@gmail.com>
Parts:
- MIC1, MIC2, MIC3, MIC4, MIC5, MIC6, MIC7, MIC8: footprint Discret:BUZ3-5 -> Capacitors_Elko_ThroughHole:Elko_vert_20x10mm_RM2.5_CopperClear
Changed lines of the file:
@@
 F 0 "MIC1" H 850 6350 60  0000 C CNN
 F 1 "ELECTRET" H 850 5850 60  0000 C CNN
-F 2 "Discret:BUZ3-5" H 750 6100 60  0001 C CNN
+F 2 "Capacitors_Elko_ThroughHole:Elko_vert_20x10mm_RM2.5_CopperClear" H 750 6100 60  0001 C CNN
 F 3 "" H 750 6100 60  0000 C CNN
 	1    850  6100
@@
 F 0 "MIC3" H 850 7850 60  0000 C CNN
 F 1 "ELECTRET" H 850 7350 60  0000 C CNN
-F 2 "Discret:BUZ3-5" H 750 7600 60  0001 C CNN
+F 2 "Capacitors_Elko_ThroughHole:Elko_vert_20x10mm_RM2.5_CopperClear" H 750 7600 60  0001 C CNN
 F 3 "" H 750 7600 60  0000 C CNN
 	1    850  7600
@@
 F 0 "MIC5" H 850 9350 60  0000 C CNN
 F 1 "ELECTRET" H 850 8850 60  0000 C CNN
-F 2 "Discret:BUZ3-5" H 750 9100 60  0001 C CNN
+F 2 "Capacitors_Elko_ThroughHole:Elko_vert_20x10mm_RM2.5_CopperClear" H 750 9100 60  0001 C CNN
 F 3 "" H 750 9100 60  0000 C CNN
 	1    850  9100
@@
 F 0 "MIC7" H 850 10850 60  0000 C CNN
 F 1 "ELECTRET" H 850 10350 60  0000 C CNN
-F 2 "Discret:BUZ3-5" H 750 10600 60  0001 C CNN
+F 2 "Capacitors_Elko_ThroughHole:Elko_vert_20x10mm_RM2.5_CopperClear" H 750 10600 60  0001 C CNN
 F 3 "" H 750 10600 60  0000 C CNN
 	1    850  10600
@@
 F 0 "MIC2" H 3050 6350 60  0000 C CNN
 F 1 "ELECTRET" H 3050 5850 60  0000 C CNN
-F 2 "Discret:BUZ3-5" H 2950 6100 60  0001 C CNN
+F 2 "Capacitors_Elko_ThroughHole:Elko_vert_20x10mm_RM2.5_CopperClear" H 2950 6100 60  0001 C CNN
 F 3 "" H 2950 6100 60  0000 C CNN
 	1    3050 6100
@@
 F 0 "MIC4" H 3050 7850 60  0000 C CNN
 F 1 "ELECTRET" H 3050 7350 60  0000 C CNN
-F 2 "Discret:BUZ3-5" H 2950 7600 60  0001 C CNN
+F 2 "Capacitors_Elko_ThroughHole:Elko_vert_20x10mm_RM2.5_CopperClear" H 2950 7600 60  0001 C CNN
 F 3 "" H 2950 7600 60  0000 C CNN
 	1    3050 7600
@@
 F 0 "MIC6" H 3050 9350 60  0000 C CNN
 F 1 "ELECTRET" H 3050 8850 60  0000 C CNN
-F 2 "Discret:BUZ3-5" H 2950 9100 60  0001 C CNN
+F 2 "Capacitors_Elko_ThroughHole:Elko_vert_20x10mm_RM2.5_CopperClear" H 2950 9100 60  0001 C CNN
 F 3 "" H 2950 9100 60  0000 C CNN
 	1    3050 9100
@@
 F 0 "MIC8" H 3050 10850 60  0000 C CNN
 F 1 "ELECTRET" H 3050 10350 60  0000 C CNN
-F 2 "Discret:BUZ3-5" H 2950 10600 60  0001 C CNN
+F 2 "Capacitors_Elko_ThroughHole:Elko_vert_20x10mm_RM2.5_CopperClear" H 2950 10600 60  0001 C CNN
 F 3 "" H 2950 10600 60  0000 C CNN
 	1    3050 10600

Commit message: Erase SPI remaining net labels and fix unconnected pins error in schematics.
Signed-off-by: Chamon <[luizchamon@gmail.com>
Connections:
- net labels removed: SPI0_CLK, SPI0_CS, SPI0_MISO, SPI0_MOSI
- wire segments 234 -> 230
- no-connect marks 76 -> 81
Changed lines of the file:
@@
 NoConn ~ 11050 5750
 NoConn ~ 11050 5850
-Text Label 10600 1700 0    60   ~ 0
-SPI0_CS
-Text Label 10500 4650 0    60   ~ 0
-SPI0_MOSI
 $Comp
 L BEAGLEBONEBLACK U2
@@
 	1    0    0    -1
 $EndComp
-Text Label 10500 1900 0    60   ~ 0
-SPI0_MISO
-Text Label 10500 4850 0    60   ~ 0
-SPI0_CLK
 Wire Wire Line
 	12900 5850 12450 5850
@@
 Wire Wire Line
 	11050 5950 10950 5950
-Wire Wire Line
-	11050 1700 10600 1700
-Wire Wire Line
-	11050 4650 10500 4650
-Wire Wire Line
-	11050 1900 10500 1900
-Wire Wire Line
-	11050 4850 10500 4850
 Text Label 8600 950  2    60   ~ 0
 PRU1_4
@@
 Wire Wire Line
 	8150 1300 8600 1300
+NoConn ~ 11050 1700
+NoConn ~ 11050 1900
+NoConn ~ 12900 2800
+NoConn ~ 11050 4650
+NoConn ~ 11050 4850
 $EndSCHEMATC

Commit message: Unify drill sizes (all drilling in 0.8 mm).
Signed-off-by: Chamon <[luizchamon@gmail.com>
Parts:
- MIC1, MIC2, MIC3, MIC4, MIC5, MIC6, MIC7, MIC8: footprint Capacitors_Elko_ThroughHole:Elko_vert_20x10mm_RM2.5_CopperClear -> micarray:Electret_1mm
- P1: footprint Pin_Headers:Pin_Header_Straight_1x03 -> micarray:Pin_Header_01x03
Changed lines of the file:
@@
 F 0 "MIC1" H 850 6350 60  0000 C CNN
 F 1 "ELECTRET" H 850 5850 60  0000 C CNN
-F 2 "Capacitors_Elko_ThroughHole:Elko_vert_20x10mm_RM2.5_CopperClear" H 750 6100 60  0001 C CNN
+F 2 "micarray:Electret_1mm" H 750 6100 60  0001 C CNN
 F 3 "" H 750 6100 60  0000 C CNN
 	1    850  6100
@@
 F 0 "MIC3" H 850 7850 60  0000 C CNN
 F 1 "ELECTRET" H 850 7350 60  0000 C CNN
-F 2 "Capacitors_Elko_ThroughHole:Elko_vert_20x10mm_RM2.5_CopperClear" H 750 7600 60  0001 C CNN
+F 2 "micarray:Electret_1mm" H 750 7600 60  0001 C CNN
 F 3 "" H 750 7600 60  0000 C CNN
 	1    850  7600
@@
 F 0 "MIC5" H 850 9350 60  0000 C CNN
 F 1 "ELECTRET" H 850 8850 60  0000 C CNN
-F 2 "Capacitors_Elko_ThroughHole:Elko_vert_20x10mm_RM2.5_CopperClear" H 750 9100 60  0001 C CNN
+F 2 "micarray:Electret_1mm" H 750 9100 60  0001 C CNN
 F 3 "" H 750 9100 60  0000 C CNN
 	1    850  9100
@@
 F 0 "MIC7" H 850 10850 60  0000 C CNN
 F 1 "ELECTRET" H 850 10350 60  0000 C CNN
-F 2 "Capacitors_Elko_ThroughHole:Elko_vert_20x10mm_RM2.5_CopperClear" H 750 10600 60  0001 C CNN
+F 2 "micarray:Electret_1mm" H 750 10600 60  0001 C CNN
 F 3 "" H 750 10600 60  0000 C CNN
 	1    850  10600
@@
 F 0 "MIC2" H 3050 6350 60  0000 C CNN
 F 1 "ELECTRET" H 3050 5850 60  0000 C CNN
-F 2 "Capacitors_Elko_ThroughHole:Elko_vert_20x10mm_RM2.5_CopperClear" H 2950 6100 60  0001 C CNN
+F 2 "micarray:Electret_1mm" H 2950 6100 60  0001 C CNN
 F 3 "" H 2950 6100 60  0000 C CNN
 	1    3050 6100
@@
 F 0 "MIC4" H 3050 7850 60  0000 C CNN
 F 1 "ELECTRET" H 3050 7350 60  0000 C CNN
-F 2 "Capacitors_Elko_ThroughHole:Elko_vert_20x10mm_RM2.5_CopperClear" H 2950 7600 60  0001 C CNN
+F 2 "micarray:Electret_1mm" H 2950 7600 60  0001 C CNN
 F 3 "" H 2950 7600 60  0000 C CNN
 	1    3050 7600
@@
 F 0 "MIC6" H 3050 9350 60  0000 C CNN
 F 1 "ELECTRET" H 3050 8850 60  0000 C CNN
-F 2 "Capacitors_Elko_ThroughHole:Elko_vert_20x10mm_RM2.5_CopperClear" H 2950 9100 60  0001 C CNN
+F 2 "micarray:Electret_1mm" H 2950 9100 60  0001 C CNN
 F 3 "" H 2950 9100 60  0000 C CNN
 	1    3050 9100
@@
 F 0 "MIC8" H 3050 10850 60  0000 C CNN
 F 1 "ELECTRET" H 3050 10350 60  0000 C CNN
-F 2 "Capacitors_Elko_ThroughHole:Elko_vert_20x10mm_RM2.5_CopperClear" H 2950 10600 60  0001 C CNN
+F 2 "micarray:Electret_1mm" H 2950 10600 60  0001 C CNN
 F 3 "" H 2950 10600 60  0000 C CNN
 	1    3050 10600
@@
 F 0 "P1" H 1050 3500 50  0000 C CNN
 F 1 "CONN_01X03" V 1150 3300 50  0001 C CNN
-F 2 "Pin_Headers:Pin_Header_Straight_1x03" H 1050 3300 60  0001 C CNN
+F 2 "micarray:Pin_Header_01x03" H 1050 3300 60  0001 C CNN
 F 3 "" H 1050 3300 60  0000 C CNN
 	1    1050 3300

Commit message: Update tantalum capacitor (C11) package.
Signed-off-by: Chamon <luizchamon@gmail.com>
Parts:
- C11: footprint Capacitors_SMD:C_0805_HandSoldering -> Capacitors_Tantalum_SMD:TantalC_SizeB_EIA-3528_HandSoldering; symbol C -> CP1
Changed lines of the file:
@@
 $EndComp
 $Comp
-L C C11
+L CP1 C11
 U 1 1 5565549D
 P 4350 2200
 F 0 "C11" H 4375 2300 50  0000 L CNN
 F 1 "22uF" H 4375 2100 50  0000 L CNN
-F 2 "Capacitors_SMD:C_0805_HandSoldering" H 4388 2050 30  0001 C CNN
+F 2 "Capacitors_Tantalum_SMD:TantalC_SizeB_EIA-3528_HandSoldering" H 4388 2050 30  0001 C CNN
 F 3 "" H 4350 2200 60  0000 C CNN
 	1    4350 2200

Commit message: Remove test point and add header on PRU pins.
Signed-off-by: Chamon <luizchamon@gmail.com>
Parts:
- removed TP1: TESTPOINT, Measurement_Points:Measurement_Point_Round-SMD-Pad_Big, symbol TESTPOINT
- added P2, P3, P4, P5, P6, P7, P8: CONN_01X02, micarray:Pin_Header_01x02, symbol CONN_01X02
Connections:
- wire segments 230 -> 250
- no-connect marks 81 -> 82
Changed lines of the file:
@@
 L DVDD #PWR021
 U 1 1 55663306
-P 8650 1800
-F 0 "#PWR021" H 8650 1650 50  0001 C CNN
-F 1 "DVDD" H 8650 1950 50  0000 C CNN
-F 2 "" H 8650 1800 60  0000 C CNN
-F 3 "" H 8650 1800 60  0000 C CNN
-	1    8650 1800
-	1    0    0    -1
-$EndComp
-$Comp
-L TESTPOINT TP1
-U 1 1 556642CA
-P 8250 1750
-F 0 "TP1" H 8500 1750 40  0000 C CNN
-F 1 "TESTPOINT" H 8300 1650 40  0001 C CNN
-F 2 "Measurement_Points:Measurement_Point_Round-SMD-Pad_Big" H 8450 1750 60  0001 C CNN
-F 3 "" H 8450 1750 60  0000 C CNN
-	1    8250 1750
+P 8600 1800
+F 0 "#PWR021" H 8600 1650 50  0001 C CNN
+F 1 "DVDD" H 8600 1950 50  0000 C CNN
+F 2 "" H 8600 1800 60  0000 C CNN
+F 3 "" H 8600 1800 60  0000 C CNN
+	1    8600 1800
 	1    0    0    -1
 $EndComp
@@
 	600  5000 6800 5000
 Wire Wire Line
-	8650 1800 8650 1950
-Wire Wire Line
-	8650 1850 8150 1850
-Wire Wire Line
-	8150 1750 8250 1750
-Wire Wire Line
-	8650 1950 8150 1950
-Connection ~ 8650 1850
+	8600 1800 8600 1950
+Wire Wire Line
+	8600 1850 8150 1850
+Wire Wire Line
+	8600 1950 8150 1950
+Connection ~ 8600 1850
 Wire Wire Line
 	10600 900  11050 900
@@
 Wire Wire Line
 	11050 5950 10950 5950
-Text Label 8600 950  2    60   ~ 0
+Text Label 9050 850  0    60   ~ 0
 PRU1_4
-Text Label 8600 1050 2    60   ~ 0
+Text Label 9050 1250 0    60   ~ 0
 PRU1_1
-Text Label 8600 1200 2    60   ~ 0
+Text Label 9050 1650 0    60   ~ 0
 PRU1_7
-Text Label 8600 1300 2    60   ~ 0
+Text Label 9050 2050 0    60   ~ 0
 PRU1_5
-Text Label 8600 1400 2    60   ~ 0
+Text Label 9050 2450 0    60   ~ 0
 PRU1_0
-Text Label 8600 1500 2    60   ~ 0
+Text Label 9050 2850 0    60   ~ 0
 PRU1_3
-Text Label 8600 2050 2    60   ~ 0
+Text Label 9050 3250 0    60   ~ 0
 PRU1_2
 Wire Wire Line
-	8150 950  8600 950
-Wire Wire Line
-	8150 1050 8600 1050
-Wire Wire Line
-	8150 1200 8600 1200
-Wire Wire Line
-	8150 1400 8600 1400
-Wire Wire Line
-	8150 1500 8600 1500
-Wire Wire Line
-	8600 2050 8150 2050
+	8150 950  8950 950
+Wire Wire Line
+	8150 1050 9300 1050
+Wire Wire Line
+	8150 1200 8950 1200
+Wire Wire Line
+	8150 1400 8850 1400
+Wire Wire Line
+	8150 1500 8800 1500
+Wire Wire Line
+	8150 2050 8750 2050
 $Comp
 L ELECTRET MIC1
@@
 	6900 550  9900 550
 Wire Notes Line
-	6900 2600 9900 2600
-Wire Notes Line
-	6900 2600 6900 550
-Text Notes 9850 2550 2    60   ~ 0
+	6900 3650 9900 3650
+Wire Notes Line
+	6900 3650 6900 550
+Text Notes 9850 3600 2    60   ~ 0
 ADC digital interface
 Text Label 10650 3950 0    60   ~ 0
@@
 Place capacitors as close as possible to BBB headers.
 Wire Notes Line
-	9900 2600 9900 550
+	9900 3650 9900 550
 NoConn ~ 700  1550
 NoConn ~ 700  1650
@@
 	12450 5750 12900 5750
 Wire Wire Line
-	8150 1300 8600 1300
+	8150 1300 8900 1300
 NoConn ~ 11050 1700
 NoConn ~ 11050 1900
@@
 NoConn ~ 11050 4650
 NoConn ~ 11050 4850
+$Comp
+L CONN_01X02 P2
+U 1 1 55AEE9A1
+P 9600 800
+F 0 "P2" H 9600 950 50  0000 C CNN
+F 1 "CONN_01X02" H 9600 650 50  0000 C CNN
+F 2 "micarray:Pin_Header_01x02" H 9600 800 60  0001 C CNN
+F 3 "" H 9600 800 60  0000 C CNN
+	1    9600 800
+	1    0    0    -1
+$EndComp
+$Comp
+L CONN_01X02 P3
+U 1 1 55AF0668
+P 9600 1200
+F 0 "P3" H 9600 1350 50  0000 C CNN
+F 1 "CONN_01X02" H 9600 1050 50  0000 C CNN
+F 2 "micarray:Pin_Header_01x02" H 9600 1200 60  0001 C CNN
+F 3 "" H 9600 1200 60  0000 C CNN
+	1    9600 1200
+	1    0    0    -1
+$EndComp
+$Comp
+L CONN_01X02 P4
+U 1 1 55AF073E
+P 9600 1600
+F 0 "P4" H 9600 1750 50  0000 C CNN
+F 1 "CONN_01X02" H 9600 1450 50  0000 C CNN
+F 2 "micarray:Pin_Header_01x02" H 9600 1600 60  0001 C CNN
+F 3 "" H 9600 1600 60  0000 C CNN
+	1    9600 1600
+	1    0    0    -1
+$EndComp
+$Comp
+L CONN_01X02 P5
+U 1 1 55AF0A11
+P 9600 2000
+F 0 "P5" H 9600 2150 50  0000 C CNN
+F 1 "CONN_01X02" H 9600 1850 50  0000 C CNN
+F 2 "micarray:Pin_Header_01x02" H 9600 2000 60  0001 C CNN
+F 3 "" H 9600 2000 60  0000 C CNN
+	1    9600 2000
+	1    0    0    -1
+$EndComp
+$Comp
+L CONN_01X02 P6
+U 1 1 55AF0CAA
+P 9600 2400
+F 0 "P6" H 9600 2550 50  0000 C CNN
+F 1 "CONN_01X02" H 9600 2250 50  0000 C CNN
+F 2 "micarray:Pin_Header_01x02" H 9600 2400 60  0001 C CNN
+F 3 "" H 9600 2400 60  0000 C CNN
+	1    9600 2400
+	1    0    0    -1
+$EndComp
+$Comp
+L CONN_01X02 P7
+U 1 1 55AF0D89
+P 9600 2800
+F 0 "P7" H 9600 2950 50  0000 C CNN
+F 1 "CONN_01X02" H 9600 2650 50  0000 C CNN
+F 2 "micarray:Pin_Header_01x02" H 9600 2800 60  0001 C CNN
+F 3 "" H 9600 2800 60  0000 C CNN
+	1    9600 2800
+	1    0    0    -1
+$EndComp
+$Comp
+L CONN_01X02 P8
+U 1 1 55AF0F49
+P 9600 3200
+F 0 "P8" H 9600 3350 50  0000 C CNN
+F 1 "CONN_01X02" H 9600 3050 50  0000 C CNN
+F 2 "micarray:Pin_Header_01x02" H 9600 3200 60  0001 C CNN
+F 3 "" H 9600 3200 60  0000 C CNN
+	1    9600 3200
+	1    0    0    -1
+$EndComp
+Wire Wire Line
+	8950 950  8950 750
+Wire Wire Line
+	8950 750  9400 750
+Wire Wire Line
+	9400 850  9050 850
+Wire Wire Line
+	9050 3250 9400 3250
+Wire Wire Line
+	9050 2850 9400 2850
+Wire Wire Line
+	9050 2450 9400 2450
+Wire Wire Line
+	9050 2050 9400 2050
+Wire Wire Line
+	9050 1650 9400 1650
+Wire Wire Line
+	9400 1250 9050 1250
+Wire Wire Line
+	9300 1050 9300 1150
+Wire Wire Line
+	9300 1150 9400 1150
+Wire Wire Line
+	8950 1200 8950 1550
+Wire Wire Line
+	8950 1550 9400 1550
+Wire Wire Line
+	8900 1300 8900 1950
+Wire Wire Line
+	8900 1950 9400 1950
+Wire Wire Line
+	8850 1400 8850 2350
+Wire Wire Line
+	8850 2350 9400 2350
+Wire Wire Line
+	8800 1500 8800 2750
+Wire Wire Line
+	8800 2750 9400 2750
+Wire Wire Line
+	8750 2050 8750 3150
+Wire Wire Line
+	8750 3150 9400 3150
+NoConn ~ 8150 1750
 $EndSCHEMATC
