File: proto_array.sch (KiCad schematic (older format))
At the start: 61 parts, among them P1 CONN_01X03, P2 CONN_01X02, P3 CONN_01X02, P4 CONN_01X02, P5 CONN_01X02, P6 CONN_01X02, P7 CONN_01X02, P8 CONN_01X02, U1 ADS131E08, U2 BEAGLEBONEBLACK

Commit message: Include switch for SYSBOOT pins and fix mic powering.
Signed-off-by: Chamon <luizchamon@gmail.com>
Parts:
- added C36, C37: 1uF, Capacitors_SMD:C_0805_HandSoldering, symbol C
- added R10, R11, R12, R13, R14, R15, R16, R9: 10k, Resistors_SMD:R_0805_HandSoldering, symbol R
- added U3: 741G04, symbol 741G04
- added U4: 743245, symbol 743245
- added U5: TLV70233DBV, symbol TLV70233DBV
Connections:
- net AGND: now also C22.1, C23.1, C26.1, C27.1, C30.1, C31.1, C34.1, C35.1, C36.2, C37.2, U3.3 (GND), U4.10 (GND), U5.2 (GND)
- net AVDD: now also C36.1, U5.1 (IN); no longer C20.1, C21.1, C24.1, C25.1, C28.1, C29.1, C32.1, C33.1, R1.1, R2.1, R3.1, R4.1, R5.1, R6.1, R7.1, R8.1
- net DVDD: now also U3.5 (VCC), U4.20 (VCC)
- net MIC_1: now also C22.2, R9.1; no longer C22.1
- net MIC_2: now also C23.2, R10.1; no longer C23.1
- net MIC_3: now also C26.2, R11.1; no longer C26.1
- net MIC_4: now also C27.2, R12.1; no longer C27.1
- net MIC_5: now also C30.2, R13.1; no longer C30.1
- net MIC_6: now also C31.2, R14.1; no longer C31.1
- net MIC_7: now also C34.2, R15.1; no longer C34.1
- net MIC_8: now also C35.2, R16.1; no longer C35.1
- net PRU1_0: now also U4.14 (B5); no longer P6.2 (P2)
- net PRU1_1: now also U4.17 (B2); no longer P3.2 (P2)
- net PRU1_2: now also U4.12 (B7); no longer P8.2 (P2)
- net PRU1_3: now also U4.13 (B6); no longer P7.2 (P2)
- net PRU1_4: now also U4.18 (B1); no longer P2.2 (P2)
- net PRU1_5: now also U4.15 (B4); no longer P5.2 (P2)
- net PRU1_7: now also U4.16 (B3); no longer P4.2 (P2)
- net PRU1_6: now reaches U2.B39 (GPIO2_12)
- net PRU1_6: now also U4.11 (B8)
- net SYS_RESETn: now reaches U2.C10 (SYS_RESETn)
- net SYS_RESETn: now also U3.2 (A)
- net at MIC1.1 (+), R1.2: now also R9.2; no longer C22.2
- net at MIC3.1 (+), R3.2: now also R11.2; no longer C26.2
- net at MIC5.1 (+), R5.2: now also R13.2; no longer C30.2
- net at MIC7.1 (+), R7.2: now also R15.2; no longer C34.2
- net at MIC2.1 (+), R2.2: now also R10.2; no longer C23.2
- net at MIC4.1 (+), R4.2: now also R12.2; no longer C27.2
- net at MIC6.1 (+), R6.2: now also R14.2; no longer C31.2
- net at MIC8.1 (+), R8.2: now also R16.2; no longer C35.2
- new net: P2.2 (P2), U4.2 (A1)
- new net: P3.2 (P2), U4.3 (A2)
- new net: P4.2 (P2), U4.4 (A3)
- new net: P5.2 (P2), U4.5 (A4)
- new net: P6.2 (P2), U4.6 (A5)
- new net: P7.2 (P2), U4.7 (A6)
- new net: P8.2 (P2), U4.8 (A7)
- new net: U3.4 (Y), U4.19 (/OE)
- new net +3V3: C20.1, C21.1, C24.1, C25.1, C28.1, C29.1, C32.1, C33.1, C37.1, R1.1, R2.1, R3.1, R4.1, R5.1, R6.1, R7.1, R8.1, U5.5 (OUT)
- new net MIC_EN: U4.9 (A8), U5.3 (EN)
- no-connect marks 82 -> 80
Other:
- note added: "Place capacitors as close as\npossible to BBB headers."
- note added: "The whole BBB draws around 200mA (460mA max,\nduring boot up). When powered by USB, the total\ncurrent drawn from the headers should probably\nnot exceed 200mA."
- note added: "VDD_3V3B comes from an LDO and is limited to 500mA.\nBBB uses this rail to power the JTAG, serial UART interface,\nLAN interface (60mA), DDR memory (80mA), and a few\npull-up resistors. DVDD should not exceed 250mA (as per SRM).\n"
- note removed: "ERC warnings relative to power output pins\nbeing connected to bidirectional pins on the\nBBB headers can safely be ignored."
- note removed: "Place capacitors as close as possible to BBB headers."
- note removed: "The whole BBB draws around 430mA (460mA max).\nWhen powered by USB, the total current drawn from\nthe headers should probably not exceed 50mA."
- note removed: "VDD_3V3B comes from an LDO and is limited to 500mA.\nBBB uses this rail to power the JTAG, serial UART interface,\nLAN interface (60mA), DDR memory (80mA), and a few\npull-up resistors. DVDD should probably not exceed 100mA.\n"
- moved on the sheet: C18, C19, C20, C21, C22, C23, C24, C25, C26, C27, C28, C29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

Commit message: Update footprints in the schematics.
Signed-off-by: Chamon <luizchamon@gmail.com>
Parts:
- added R17, R18, R19, R20, R21, R22, R23, R24: NI, Resistors_SMD:R_0805_HandSoldering, symbol R
- P2, P3, P4, P5, P6, P7, P8: footprint micarray:Pin_Header_01x02 -> micarray:Pin_Header_NC_01x02
- U3: footprint (none) -> micarray:SOTFL-5_160x50_Pitch0.5
- U4: footprint (none) -> micarray:SOP-20_600x175_Pitch0.635
- U5: footprint (none) -> micarray:SOT-23-5
Connections:
- net MIC_EN: now also R24.2
- net PRU1_0: now also R21.1
- net PRU1_1: now also R18.1
- net PRU1_2: now also R23.1
- net PRU1_3: now also R22.1
- net PRU1_4: now also R17.1
- net PRU1_5: now also R20.1
- net PRU1_6: now also R24.1
- net PRU1_7: now also R19.1
- net ADS_START: now reaches P2.2 (P2), U4.2 (A1)
- net ADS_START: now also R17.2
- net ADS_DRDY: now reaches P3.2 (P2), U4.3 (A2)
- net ADS_DRDY: now also R18.2
- net ADS_CS: now reaches P4.2 (P2), U4.4 (A3)
- net ADS_CS: now also R19.2
- net ADS_SCLK: now reaches P5.2 (P2), U4.5 (A4)
- net ADS_SCLK: now also R20.2
- net ADS_DIN: now reaches P6.2 (P2), U4.6 (A5)
- net ADS_DIN: now also R21.2
- net ADS_DOUT: now reaches P7.2 (P2), U4.7 (A6)
- net ADS_DOUT: now also R22.2
- net ADS_RESET: now reaches P8.2 (P2), U4.8 (A7)
- net ADS_RESET: now also R23.2
Other:
- note added: "These SMD jumpers can be used\nto bypass the SN743245 if it\nposes any problem."
- note added: "These jumpers are normally connected\nand only need to be installed if there\nis a problem with the SN743245."
- moved on the sheet: C20, C21, C22, C23, C24, C25, C26, C27, C28, C29, C30, C31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

Commit message: Remove NI resistors and include jumper between GNDs.
Signed-off-by: Chamon <luizchamon@gmail.com>
Parts:
- removed R17, R18, R19, R20, R21, R22, R23, R24: NI, Resistors_SMD:R_0805_HandSoldering, symbol R
- added JP1: JUMPER, micarray:Jumper, symbol JUMPER
Connections:
- net ADS_CS: now also U1.39 (/CS), U4.5 (A4); no longer P4.2 (P2), U4.4 (A3)
- net ADS_DIN: now also U1.34 (DIN), U4.8 (A7); no longer P6.2 (P2), U4.6 (A5)
- net ADS_DOUT: now also U1.43 (DOUT), U4.3 (A2); no longer P7.2 (P2), U4.7 (A6)
- net ADS_DRDY: now also U1.47 (/DRDY), U4.2 (A1); no longer P3.2 (P2), U4.3 (A2)
- net ADS_RESET: now also U1.36 (/RESET), U4.7 (A6); no longer P8.2 (P2), U4.8 (A7)
- net ADS_SCLK: now also U1.40 (SCLK), U4.4 (A3); no longer P5.2 (P2), U4.5 (A4)
- net ADS_START: now also U1.38 (START), U4.6 (A5); no longer P2.2 (P2), U4.2 (A1)
- net AGND: now also JP1.1; no longer C1.2, C19.2, C2.2, U1.31 (RESV1), U1.33 (DGND), U1.49 (DGND), U1.51 (DGND), U2.B1 (DGND), U2.B2 (DGND), U2.C43 (DGND), U2.C44 (DGND), U3.3 (GND), U4.10 (GND)
- net AVDD: now also U5.3 (EN)
- net PRU1_0: now also P6.2 (P2); no longer U4.14 (B5)
- net PRU1_1: now also P3.2 (P2); no longer U4.17 (B2)
- net PRU1_2: now also P8.2 (P2); no longer U4.12 (B7)
- net PRU1_3: now also P7.2 (P2); no longer U4.13 (B6)
- net PRU1_4: now also P2.2 (P2); no longer U4.18 (B1)
- net PRU1_5: now also P5.2 (P2); no longer U4.15 (B4)
- net PRU1_7: now also P4.2 (P2); no longer U4.16 (B3)
- net at P6.1 (P1): now also U4.12 (B7); no longer U1.34 (DIN)
- net at P8.1 (P1): now also U4.13 (B6); no longer U1.36 (/RESET)
- net at P2.1 (P1): now also U4.14 (B5); no longer U1.38 (START)
- net at P4.1 (P1): now also U4.15 (B4); no longer U1.39 (/CS)
- net at P5.1 (P1): now also U4.16 (B3); no longer U1.40 (SCLK)
- net at P7.1 (P1): now also U4.17 (B2); no longer U1.43 (DOUT)
- net at P3.1 (P1): now also U4.18 (B1); no longer U1.47 (/DRDY)
- net MIC_EN: no longer names the net of U4.9 (A8)
- net MIC_EN: no longer U5.3 (EN)
- net PRU1_6: no longer names the net of U2.B39 (GPIO2_12)
- net PRU1_6: no longer U4.11 (B8)
- new net DGND: C1.2, C19.2, C2.2, JP1.2, U1.31 (RESV1), U1.33 (DGND), U1.49 (DGND), U1.51 (DGND), U2.B1 (DGND), U2.B2 (DGND), U2.C43 (DGND), U2.C44 (DGND), U3.3 (GND), U4.10 (GND)
Other:
- note removed: "These SMD jumpers can be used\nto bypass the SN743245 if it\nposes any problem."
- moved on the sheet: P2, P3, P4, P5, P6, P7, P8, U2A, U2B, U2C, U2D, U3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

Commit message: Add bypass to 743245 and fix pinout of 741G04.
Signed-off-by: Chamon <luizchamon@gmail.com>
Parts:
- added C38: 1uF, Capacitors_SMD:C_0805_HandSoldering, symbol C
Connections:
- net AGND: no longer C14.2, C15.2
- net DGND: now also C14.2, C15.2, C38.2
- net DVDD: now also C38.1
- no-connect marks 80 -> 83
Other:
- note added: "Place capacitors\nas close as possible\nto BBB headers."
- note removed: "Place capacitors as close as\npossible to BBB headers."
- moved on the sheet: C37, P2, P3, P4, P5, P6, P7, P8, U4

Commit message: Fix issue with TLV schematic symbol.
Signed-off-by: Chamon <luizchamon@gmail.com>
Parts:
- U5: symbol TLV70233DBV -> TLV70233DBV-2
Connections:
- net AGND: now also U5.4 (NC)
Changed lines of the file:
@@
 EESchema Schematic File Version 2
+LIBS:proto_array-rescue
 LIBS:power
 LIBS:device
@@
 $EndComp
 $Comp
-L TLV70233DBV U5
+L TLV70233DBV-2 U5
 U 1 1 55B9C715
 P 1550 4150
